File: Logic_Board_1A/LB1A_DCA7M4_R512MB_F4GB/Design/Rev_1.0.0/Kicad/LB1A_DCA7M4_R512MB_F4GB.kicad_pcb (KiCad board)
At the start: 6 copper layers, 50 x 50 mm, 143 parts, among them U1 STM32MP157CAC3, U2 AS4C256M16D3LC-12BCN, U3 S40FC004C1B2C00000, U4 STPMIC1BPQR, U5 DF40C-70DP-0.4V(51), U6 DF40C-70DP-0.4V(51), U7 DF40C-70DP-0.4V(51), X1 32.768kHz, X2 24MHz

Commit message: improvements on sch and pcb
Parts:
- R2: moved to B.Cu
- moved C2 0.19 mm to (138.6, 98.7)
- moved C5 0.15 mm to (138.6, 97.7)
Connections:
- C38 pad 1: PMIC_VOUT3_VDD -> PMIC_LDO5_2V9
- C39 pad 1: PMIC_VOUT3_VDD -> PMIC_LDO5_2V9
- C40 pad 1: PMIC_VOUT3_VDD -> PMIC_LDO5_2V9
- C41 pad 1: PMIC_VOUT3_VDD -> PMIC_LDO5_2V9
- C60 pad 1: PMIC_LDO5 -> PMIC_LDO5_2V9
- R36 pad 1: PMIC_VOUT3_VDD -> PMIC_LDO5_2V9
- R37 pad 1: PMIC_VOUT3_VDD -> PMIC_LDO5_2V9
- R38 pad 1: PMIC_VOUT3_VDD -> PMIC_LDO5_2V9
- R39 pad 1: PMIC_VOUT3_VDD -> PMIC_LDO5_2V9
- R40 pad 1: PMIC_VOUT3_VDD -> PMIC_LDO5_2V9
- R41 pad 1: PMIC_VOUT3_VDD -> PMIC_LDO5_2V9
- R42 pad 1: PMIC_VOUT3_VDD -> PMIC_LDO5_2V9
- R43 pad 1: PMIC_VOUT3_VDD -> PMIC_LDO5_2V9
- R44 pad 1: PMIC_VOUT3_VDD -> PMIC_LDO5_2V9
- R45 pad 1: PMIC_VOUT3_VDD -> PMIC_LDO5_2V9
- U3 pad A9: PMIC_VOUT3_VDD -> PMIC_LDO5_2V9
- U3 pad B8: PMIC_VOUT3_VDD -> PMIC_LDO5_2V9
- U3 pad C6: PMIC_VOUT3_VDD -> PMIC_LDO5_2V9
- U3 pad C7: PMIC_VOUT3_VDD -> PMIC_LDO5_2V9
- U3 pad E6: PMIC_VOUT3_VDD -> PMIC_LDO5_2V9
- U3 pad F5: PMIC_VOUT3_VDD -> PMIC_LDO5_2V9
- U3 pad J10: PMIC_VOUT3_VDD -> PMIC_LDO5_2V9
- U3 pad K9: PMIC_VOUT3_VDD -> PMIC_LDO5_2V9
- U3 pad M4: PMIC_VOUT3_VDD -> PMIC_LDO5_2V9
- U3 pad N4: PMIC_VOUT3_VDD -> PMIC_LDO5_2V9
- U3 pad P3: PMIC_VOUT3_VDD -> PMIC_LDO5_2V9
- U3 pad P5: PMIC_VOUT3_VDD -> PMIC_LDO5_2V9
- U4 pad 20: PMIC_LDO5 -> PMIC_LDO5_2V9
- U5 pad 10: LCD_R2 -> LCD_R3
- U5 pad 12: LCD_R3 -> LCD_R2
- U5 pad 16: DSI_D0_N -> DSI_TE
- U5 pad 18: DSI_TE -> DSI_D0_N
- U5 pad 25: U_LED_1 -> BOOT1
- U5 pad 34: JTMS_SWDIO -> DSI_RESET
- U5 pad 35: BOOT1 -> U_LED_1
- U5 pad 36: DSI_RESET -> JTMS_SWDIO
- U6 pad 51: PMIC_LDO5 -> PMIC_LDO5_2V9
- U6 pad 53: PMIC_LDO5 -> PMIC_LDO5_2V9
- U7 pad 32: LCD_R5 -> ETH_CLK125
- U7 pad 34: ETH_CLK125 -> LCD_R5
- U7 pad 47: ETH_TXD0 -> I2C1_SDA
- U7 pad 49: I2C1_SDA -> ETH_TXD0
- U7 pad 50: Net-(U7-Pad50) -> LCD_DE
- U7 pad 52: Net-(U7-Pad52) -> SPI5_MISO
- U7 pad 54: LCD_DE -> LCD_B2
- U7 pad 56: SPI5_MISO -> Net-(U7-Pad56)
- U7 pad 58: LCD_B2 -> Net-(U7-Pad58)
- U7 pad 64: Net-(U7-Pad64) -> SPI5_NSS
- U7 pad 66: SPI5_NSS -> LCD_CLK
- U7 pad 68: LCD_CLK -> Net-(U7-Pad68)
- U7 pad 69: DSI_BL_CTRL -> USART1_RTS
- U7 pad 70: USART1_RTS -> DSI_BL_CTRL
Routing:
- net PMIC_LDO5_2V9: track 0.00 -> 68.1 mm, vias 0 -> 12
- net PMIC_LDO5: track 46.4 -> 0.00 mm, vias 3 -> 0
- net PMIC_VOUT3_VDD: track 67.9 -> 47.4 mm, vias 32 -> 23
- net I2C4_SCL: track 73.3 -> 82.5 mm
- net I2C4_SDA: track 77.0 -> 84.7 mm
- net GND: track 200.3 -> 206.0 mm, vias 137 -> 133
- net PMIC_WAKEUP: track 46.7 -> 51.9 mm
- net U_LED_1: track 57.4 -> 62.4 mm
- net LCD_B0: track 50.8 -> 55.4 mm
- net LCD_G7: track 50.5 -> 55.1 mm
- net I2S2_SDO: track 48.7 -> 53.3 mm
- net LCD_R2: track 32.6 -> 37.0 mm
- net LCD_G2: track 48.7 -> 44.5 mm
- net LCD_G6: track 50.9 -> 54.8 mm
- net LCD_R3: track 33.0 -> 36.8 mm
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- added copper zone on Signal_Layer_3.Cu, net PMIC_LDO5_2V9
Other:
- net class DDR_DiffPairs: clearance 0.08 -> 0.1016; trace_width 0.09 -> 0.0889; via_dia 0.4 -> 0.40005; via_drill 0.2 -> 0.20066
- net class Default: clearance 0.08 -> 0.1016; trace_width 0.09 -> 0.0889; via_dia 0.4 -> 0.40005; via_drill 0.2 -> 0.20066
- net class Gnd_Lines added: clearance 0.1016, trace_width 0.2032, via_dia 0.40005, via_drill 0.20066
- rule trace_clearance: 0.08 -> 0.1016
- rule trace_min: 0.09 -> 0.0889
- rule via_min_drill: 0.2 -> 0.20066
- rule via_min_size: 0.4 -> 0.40005

Commit message: some more improvements
Routing:
- net LCD_G2: track 44.5 -> 52.3 mm
- net LCD_R6: track 48.6 -> 52.6 mm
- net LCD_G5: track 46.8 -> 50.5 mm
- net STLINK_UART4_TX: track 43.3 -> 47.0 mm
- net LCD_R4: track 48.7 -> 52.3 mm
- net LCD_B3: track 41.0 -> 44.5 mm
- net LCD_G4: track 46.5 -> 49.9 mm
- net LCD_G3: track 40.8 -> 44.1 mm
- net LCD_R7: track 40.9 -> 44.1 mm
- net I2S2_WS: track 42.0 -> 44.2 mm, vias 1 -> 2
- net LCD_G1: track 45.1 -> 47.2 mm, vias 1 -> 2
- net STLINK_UART4_RX: track 40.8 -> 42.8 mm, vias 1 -> 2
- net LCD_B4: track 39.0 -> 40.8 mm, vias 1 -> 2
- net LCD_B0: track 55.4 -> 54.9 mm

Commit message: more improvements
Parts:
- C38, C42, R41, R42, R44, R45: moved to B.Cu
Connections:
- U5 pad 34: DSI_RESET -> JTMS_SWDIO
- U5 pad 36: JTMS_SWDIO -> DSI_RESET
Routing:
- net PMIC_LDO5_2V9: track 68.1 -> 63.4 mm, vias 12 -> 10
- net DSI_CKP: track 33.2 -> 37.5 mm
- net Net-(C42-Pad1): track 3.44 -> 0.50 mm
- net SDMMC2_D6: track 24.4 -> 26.3 mm
- net SDMMC2_D5: track 20.6 -> 22.4 mm
- net DSI_D0_P: track 33.0 -> 34.8 mm
- net SDMMC2_CK: track 30.5 -> 32.3 mm
- net DSI_CKN: track 33.8 -> 35.5 mm
- net DSI_D1_N: track 34.4 -> 35.8 mm
- net DSI_D1_P: track 33.7 -> 35.2 mm
- net GND: track 206.0 -> 204.7 mm, vias 133 -> 131
- net JTDO_TRACESWO: track 34.7 -> 35.4 mm
- net DSI_RESET: track 29.6 -> 30.2 mm

Commit message: Improvements to PCB
Routing:
- net DDR_DQ3: track 24.7 -> 35.3 mm
- net DDR_DQ5: track 26.2 -> 34.4 mm
- net DDR_DQ0: track 25.1 -> 32.2 mm
- net DDR_DQS0_N: track 26.5 -> 33.5 mm
- net DDR_DQ4: track 27.3 -> 34.1 mm
- net DDR_DQ1: track 25.3 -> 31.6 mm
- net DDR_DQM0: track 25.6 -> 31.6 mm
- net DDR_DQ2: track 26.1 -> 31.6 mm
- net DDR_DQ7: track 26.9 -> 32.1 mm
- net DDR_DQ6: track 27.2 -> 32.2 mm
- net DDR_DQS0_P: track 27.1 -> 31.6 mm
Other:
- net class DDR_DiffPairs: clearance 0.1016 -> 0.0762
- net class Default: clearance 0.1016 -> 0.0762
- net class Gnd_Lines: clearance 0.1016 -> 0.0762
- rule trace_clearance: 0.1016 -> 0.0762

Commit message: pcb improvements
Routing:
- net DDR_A14: track 34.8 -> 24.0 mm
- net DDR_A12: track 32.7 -> 22.9 mm
- net DDR_A11: track 32.9 -> 23.4 mm
- net DDR_A10: track 30.4 -> 22.2 mm
- net DDR_CLK_P: track 26.7 -> 18.8 mm
- net DDR_CLK_N: track 25.8 -> 18.4 mm
- net DDR_A1: track 35.1 -> 28.2 mm
- net DDR_A6: track 24.1 -> 18.7 mm
- net DDR_DQ13: track 23.1 -> 28.3 mm
- net DDR_DQ15: track 24.6 -> 29.7 mm
- net DDR_A4: track 25.1 -> 20.2 mm
- net DDR_DQ14: track 22.8 -> 27.3 mm
- net DDR_RASN: track 29.5 -> 25.5 mm
- net DDR_CASN: track 30.0 -> 26.6 mm
- net DDR_WEN: track 29.2 -> 25.9 mm
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Other:
- net class DDR_DiffPairs: clearance 0.0762 -> 0.1016
- net class Default: clearance 0.0762 -> 0.1016
- net class Gnd_Lines: clearance 0.0762 -> 0.1016
- rule trace_clearance: 0.0762 -> 0.1016
