File: Logic_Board_1D/LB1D_DCA7M4_R512MB_F4GB/Design/Kicad/Rev_1.0.0/Kicad/LB1D_DCA7M4_R512MB_F4GB.kicad_pcb (KiCad board)
At the start: 4 copper layers, 50 x 50 mm, 144 parts, among them U1 STM32MP157CAC3, U3 S40FC004C1B2C00000, U4 STPMIC1BPQR, U5 DF40C-70DP-0.4V(51), U6 DF40C-70DP-0.4V(51), U7 DF40C-70DP-0.4V(51), X1 32.768kHz, X2 24MHz

Commit message: Pcb routing
Parts:
- removed the U1 at (148.5, 94.2)
- added C32: 10uF, Capacitor_SMD:C_0402_1005Metric, F.Cu at (179.1, 106.4)
- added C33: 10pF, Capacitor_SMD:C_0402_1005Metric, F.Cu at (182.0, 106.4)
- added R47: 100E, Resistor_SMD:R_0402_1005Metric, F.Cu at (176.2, 104.9)
- added R48: 100E, Resistor_SMD:R_0402_1005Metric, F.Cu at (179.1, 104.4)
- added R49: 0E, Capacitor_SMD:C_0402_1005Metric, F.Cu at (184.8, 104.9)
- added R50: 100k, Capacitor_SMD:C_01005_0402Metric, F.Cu at (193.4, 95.2)
- added R51: 100k, Capacitor_SMD:C_01005_0402Metric, F.Cu at (193.4, 96.8)
- added R52: 100k, Capacitor_SMD:C_01005_0402Metric, F.Cu at (187.4, 104.8)
- added R53: 100k, Capacitor_SMD:C_01005_0402Metric, F.Cu at (193.4, 98.5)
- added R54: 100k, Capacitor_SMD:C_01005_0402Metric, F.Cu at (187.4, 106.4)
- added R55: 100k, Capacitor_SMD:C_01005_0402Metric, F.Cu at (193.4, 100.1)
- added TP1: TestPoint, TestPoint:TestPoint_Pad_D1.0mm, F.Cu at (173.2, 105.0)
- added U8: WFM200S022XNA3R, U_Module:WFM200S022XNA3, F.Cu at (146.8, 111.6)
- added U9: BGX220S22HNA21R, U_Module:BGX220S22HNA21, F.Cu at (121.0, 104.1)
- moved R1 3.66 mm to (142.4, 86.0)
- moved C2 2.77 mm to (138.7, 92.1)
- moved C5 2.77 mm to (138.7, 91.1)
- moved C38 2.01 mm to (128.4, 91.1)
- moved C39 2.01 mm to (138.7, 92.4)
- moved C40 2.01 mm to (138.7, 99.9)
- moved C42 2.01 mm to (135.1, 91.2)
- moved R37 2.01 mm to (138.7, 96.7)
- moved R39 2.01 mm to (138.7, 93.5)
- moved R42 2.01 mm to (133.0, 91.2)
- moved R43 2.01 mm to (138.7, 98.9)
- moved R45 2.01 mm to (130.5, 91.1)
- moved U3 2.01 mm to (132.8, 97.8)
- moved C41 2.01 mm to (127.3, 96.0)
- moved R36 2.01 mm to (138.7, 95.6)
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- renumbered Ue to U2
Connections:
- U1 pad A4: Net-(U1-PadA4) -> WIFI_IRQ
- U1 pad A5: Net-(U1-PadA5) -> SDMMC3_CMD
- U1 pad AB9: Net-(U1-PadAB9) -> USART3_RTS
- U1 pad AC10: Net-(U1-PadAC10) -> USART3_CTS
- U1 pad AC5: Net-(U1-PadAC5) -> USART3_RX
- U1 pad B3: Net-(U1-PadB3) -> WIFI_WKUP
- U1 pad B7: Net-(U1-PadB7) -> SDMMC3_CK
- U1 pad D10: Net-(U1-PadD10) -> SDMMC3_D3
- U1 pad D7: Net-(U1-PadD7) -> SDMMC3_D2
- U1 pad D8: Net-(U1-PadD8) -> SDMMC3_D0
- U1 pad D9: Net-(U1-PadD9) -> SDMMC3_D1
- U1 pad Y3: Net-(U1-PadY3) -> USART3_TX
- U1 pad Y5: Net-(U1-PadY5) -> BLE_RESET
Routing:
- net DDR_DQ0: track 0.00 -> 39.6 mm, vias 0 -> 2
- net DDR_DQS0_P: track 0.00 -> 31.6 mm, vias 0 -> 2
- net DDR_DQ7: track 0.00 -> 31.6 mm, vias 0 -> 2
- net DDR_DQ3: track 0.00 -> 31.6 mm, vias 0 -> 2
- net DDR_DQ1: track 0.00 -> 31.6 mm, vias 0 -> 2
- net DDR_DQS0_N: track 0.00 -> 31.6 mm, vias 0 -> 2
- net DDR_DQM0: track 0.00 -> 31.6 mm, vias 0 -> 2
- net DDR_A7: track 0.00 -> 26.6 mm, vias 0 -> 2
- net PMIC_VOUT2_VDD_DDR: track 0.00 -> 16.7 mm, vias 0 -> 5
- net DDR_RESETN: track 0.00 -> 15.6 mm, vias 0 -> 2
- net GND: track 0.00 -> 8.36 mm, vias 0 -> 16
- net DDR_DQ6: track 0.00 -> 7.03 mm, vias 0 -> 1
- net Net-(R1-Pad1): track 0.00 -> 6.66 mm
- net DDR_BA2: track 0.00 -> 6.00 mm, vias 0 -> 1
- net Net-(C5-Pad2): track 0.00 -> 5.60 mm, vias 0 -> 1
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- added copper zone on Signal_Layer_2.Cu, net PMIC_VOUT2_VDD_DDR
Other:
- net class DDR_DiffPairs removed
- net class Default: trace_width 0.0889 -> 0.1016

Commit message: changes
Routing:
- net DDR_DQ12: track 0.00 -> 32.0 mm
- net DDR_DQ4: track 0.00 -> 31.6 mm, vias 0 -> 2
- net DDR_DQ5: track 0.99 -> 31.6 mm, vias 1 -> 2
- net DDR_A13: track 0.00 -> 30.1 mm, vias 0 -> 2
- net DDR_DQ2: track 2.16 -> 32.1 mm, vias 1 -> 2
- net DDR_A9: track 0.00 -> 28.8 mm, vias 0 -> 2
- net DDR_DQ8: track 0.00 -> 27.8 mm
- net DDR_DQ10: track 0.00 -> 27.8 mm
- net DDR_DQ9: track 0.00 -> 27.7 mm
- net DDR_DQ13: track 0.00 -> 27.7 mm
- net DDR_DQS1_N: track 0.00 -> 27.6 mm
- net DDR_DQ15: track 0.00 -> 27.6 mm
- net DDR_DQ14: track 0.00 -> 27.6 mm
- net DDR_DQ11: track 0.00 -> 27.6 mm
- net DDR_DQM1: track 0.00 -> 27.5 mm
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